Commit message: inertias added

File: automi_description/urdf/arm.urdf.xacro (robot description, xacro)
@@ -12,6 +12,6 @@
             <inertial>
                 <origin xyz="0.0 0.0 0.0" rpy="0.0 0.0 0.0"/>
-                <mass value="1.0"/>
-                <inertia ixx="0.0" ixy="0.0" ixz="0.0" iyy="0.0" iyz="0.0" izz="0.0"/>
+                <mass value="0.0114101"/>
+                <inertia ixx="2.20572018e-06" ixy="-0" ixz="-6.183e-11" iyy="4.83772068e-06" iyz="-5.6590326e-07" izz="4.41215019e-06"/>
             </inertial>
             <visual name="">
@@ -38,6 +38,6 @@
             <inertial>
                 <origin xyz="0.0 0.0 0.0" rpy="0.0 0.0 0.0"/>
-                <mass value="1.0"/>
-                <inertia ixx="0.0" ixy="0.0" ixz="0.0" iyy="0.0" iyz="0.0" izz="0.0"/>
+                <mass value="0.0217184"/>
+                <inertia ixx="8.43192828e-06" ixy="-1.62e-12" ixz="2.16e-12" iyy="8.78536152e-06" iyz="-2.7e-12" izz="1.33461094e-05"/>
             </inertial>
             <visual name="">
@@ -66,6 +66,6 @@
             <inertial>
                 <origin xyz="0.0 0.0 0.0" rpy="0.0 0.0 0.0"/>
-                <mass value="1.0"/>
-                <inertia ixx="0.0" ixy="0.0" ixz="0.0" iyy="0.0" iyz="0.0" izz="0.0"/>
+                <mass value="0.0217184"/>
+                <inertia ixx="8.43192828e-06" ixy="-1.62e-12" ixz="2.16e-12" iyy="8.78536152e-06" iyz="-2.7e-12" izz="1.33461094e-05"/>
             </inertial>
             <visual name="">

File: automi_description/urdf/dynamixels.urdf.xacro (robot description, xacro)
@@ -29,9 +29,6 @@
             <inertial>
                 <origin xyz="0 0 0"/>
-                <mass value="0.0546"/>
-                <inertia
-                    ixx="1.57e-5" ixy="0" ixz="0"
-                    iyy="0" iyz="0"
-                    izz="0"/>
+                <mass value="0.115109"/>
+                <inertia ixx="3.3239562e-08" ixy="-1.71315e-12"ixz="7.3197e-12" iyy="1.83264787e-08" iyz="-2.8088019e-10" izz="2.79685224e-08"/>
             </inertial>
             <visual>

File: automi_description/urdf/leg.urdf.xacro (robot description, xacro)
@@ -13,6 +13,6 @@
             <inertial>
                 <origin xyz="0.0 0.0 0.0" rpy="0.0 0.0 0.0"/>
-                <mass value="1.0"/>
-                <inertia ixx="0.0" ixy="0.0" ixz="0.0" iyy="0.0" iyz="0.0" izz="0.0"/>
+                <mass value="0.0524686"/>
+                <inertia ixx="3.79355686e-05" ixy="1.22736951e-05" ixz="2.4462e-10" iyy="6.47107923e-05" iyz="2.1033e-10" izz="7.72305303e-05"/>
             </inertial>
             <visual name="">
@@ -55,6 +55,6 @@
             <inertial>
                 <origin xyz="0.0 0.0 0.0" rpy="0.0 0.0 0.0"/>
-                <mass value="1.0"/>
-                <inertia ixx="0.0" ixy="0.0" ixz="0.0" iyy="0.0" iyz="0.0" izz="0.0"/>
+                <mass value="0.0308695"/>
+                <inertia ixx="2.44928245e-05" ixy="-8.1e-13" ixz="-1.08e-12" iyy="1.5896763e-05" iyz="-1.055808e-07" izz="1.52603879e-05"/>
             </inertial>
             <visual name="">
@@ -83,6 +83,6 @@
             <inertial>
                 <origin xyz="0.0 0.0 0.0" rpy="0.0 0.0 0.0"/>
-                <mass value="1.0"/>
-                <inertia ixx="0.0" ixy="0.0" ixz="0.0" iyy="0.0" iyz="0.0" izz="0.0"/>
+                <mass value="0.0387102"/>
+                <inertia ixx="4.41099235e-05" ixy="-0" ixz="-5.4e-13" iyy="3.13463693e-05" iyz="-2.8154088e-07" izz="1.91534236e-05"/>
             </inertial>
             <visual name="">

File: automi_description/urdf/torso.urdf.xacro (robot description, xacro)
@@ -14,6 +14,6 @@
             <inertial>
                 <origin xyz="0.0 0.0 0.0" rpy="0.0 0.0 0.0"/>
-                <mass value="1.0"/>
-                <inertia ixx="0.0" ixy="0.0" ixz="0.0" iyy="0.0" iyz="0.0" izz="0.0"/>
+                <mass value="0.131665"/>
+                <inertia ixx="0.000519418268" ixy="-1.79595195e-05" ixz="1.2075507e-07" iyy="0.00048709882" iyz="3.8656764e-07" izz="0.000115698856"/>
             </inertial>
             <visual>
@@ -44,6 +44,6 @@
             <inertial>
                 <origin xyz="0.0 0.0 0.0" rpy="0.0 0.0 0.0"/>
-                <mass value="1.0"/>
-                <inertia ixx="0.0" ixy="0.0" ixz="0.0" iyy="0.0" iyz="0.0" izz="0.0"/>
+                <mass value="1.55086"/>
+                <inertia ixx="0.0034367683" ixy="5.09836432e-05" ixz="4.77030168e-06" iyy="0.00293127768" iyz="-4.57789663e-05" izz="0.00196796593"/>
             </inertial>
             <visual name="">
@@ -74,6 +74,6 @@
             <inertial>
                 <origin xyz="0.0 0.0 0.0" rpy="0.0 0.0 0.0"/>
-                <mass value="1.0"/>
-                <inertia ixx="0.0" ixy="0.0" ixz="0.0" iyy="0.0" iyz="0.0" izz="0.0"/>
+                <mass value="0.128678"/>
+                <inertia ixx="0.000284733358" ixy="-1.04236092e-06" ixz="-7.3232262e-07" iyy="0.000360225319" iyz="-6.1818174e-07" izz="0.000135432051"/>
             </inertial>
             <visual name="">
@@ -101,6 +101,6 @@
         <link name="${name}_int_head">
             <inertial>
-                <mass value="0.0005"/>
-                <inertia ixx="0.0" ixy="0.0" ixz="0.0" iyy="0.0" iyz="0.0" izz="0.0"/>
+                <mass value="0.00485437"/>
+                <inertia ixx="8.2936386e-07" ixy="0" ixz="0" iyy="1.0523979e-06" iyz="0" izz="2.7679914e-07"/>
             </inertial>
             <visual name="">
@@ -129,6 +129,6 @@
             <inertial>
                 <origin xyz="0.0 0.0 0.0" rpy="0.0 0.0 0.0"/>
-                <mass value="1.0"/>
-                <inertia ixx="0.0" ixy="0.0" ixz="0.0" iyy="0.0" iyz="0.0" izz="0.0"/>
+                <mass value="0.0197099"/>
+                <inertia ixx="3.31024347e-06" ixy="-8.1e-13" ixz="-8.1e-13" iyy="8.74277118e-06" iyz="-4.4037e-10" izz="7.77454497e-06"/>
             </inertial>
             <visual name="">
